Commit message: overhead camera positioned

File: vegebot_run/urdf/vegebot.urdf.xacro (robot description, xacro)
@@ -6,4 +6,5 @@
 -->
   <!-- Vegebot platform dimensions -->
+  <xacro:property name="MPI" value="3.14159265359" />
   <xacro:property name="floor_thickness" value="0.05" />
   <xacro:property name="platform_width" value="2.12" />
@@ -47,4 +48,13 @@
   <xacro:property name="camera_size" value="0.05" />
   <xacro:property name="camera_offset_z" value="0.03" />
+  <xacro:property name="overhead_camera_support1_length" value="1.2" />
+  <xacro:property name="overhead_camera_support1_width" value="0.045" />
+  <xacro:property name="overhead_camera_support1_height" value="0.045" />
+  <xacro:property name="overhead_camera_support2_length" value="0.88" />
+  <xacro:property name="overhead_camera_support2_width" value="0.045" />
+  <xacro:property name="overhead_camera_support2_height" value="0.045" />
+  <xacro:property name="overhead_camera_length" value="0.06" />
+  <xacro:property name="overhead_camera_width" value="0.1" />
+  <xacro:property name="overhead_camera_height" value="0.045" />
   <xacro:macro name="wheel_assembly">
     <visual>
@@ -209,4 +219,52 @@
     </visual>
   </link>
+  <link name="overhead_camera_support1">
+    <visual>
+      <geometry>
+        <box size="${overhead_camera_support1_length} ${overhead_camera_support1_width} ${overhead_camera_support1_height}" />
+      </geometry>
+      <origin xyz="-0.6 0.0 0.0" />
+      <material name="gray">
+         <color rgba="0.1 0.1 0.1 1" />
+      </material>
+    </visual>
+  </link>
+  <joint name="platform_to_overhead_camera_support1_joint" type="fixed">
+    <parent link="platform" />
+    <child link = "overhead_camera_support1" />
+    <origin xyz="${-front_platform_to_origin_arm} 0.0 ${platform_height}" rpy="0.0 ${MPI/2.0} 0.0" />
+  </joint>
+  <link name="overhead_camera_support2">
+    <visual>
+      <geometry>
+        <box size="${overhead_camera_support2_length} ${overhead_camera_support2_width} ${overhead_camera_support2_height}" />
+      </geometry>
+      <origin xyz="${-overhead_camera_support2_length/2.0} 0.0 0.0" />
+      <material name="gray">
+         <color rgba="0.1 0.1 0.1 1" />
+      </material>
+    </visual>
+  </link>
+  <joint name="overhead_camera_support1_to_overhead_camera_support2_joint" type="fixed">
+    <parent link="overhead_camera_support1" />
+    <child link = "overhead_camera_support2" />
+    <origin xyz="${-overhead_camera_support1_length + (overhead_camera_support2_width/2.0)} 0.0 ${overhead_camera_support2_width/2.0}" rpy="0.0 ${MPI/2.0} 0.0" />
+  </joint>
+  <link name="overhead_camera">
+    <visual>
+      <geometry>
+        <box size="${overhead_camera_length} ${overhead_camera_width} ${overhead_camera_height}" />
+      </geometry>
+      <origin xyz="${-overhead_camera_length/2.0} 0.0 0.0" />
+      <material name="red">
+         <color rgba="1 0 0 1" />
+      </material>
+    </visual>
+  </link>
+  <joint name="overhead_camera_support2_to_overhead_camera_joint" type="fixed">
+    <parent link="overhead_camera_support2" />
+    <child link = "overhead_camera" />
+    <origin xyz="${-overhead_camera_support2_length + (overhead_camera_height/2.0)} 0.0 ${overhead_camera_support2_height/2.0 + overhead_camera_height/2.0}" rpy="0.0 ${MPI/2.0} 0.0" />
+  </joint>
   <joint name="world_joint" type="fixed">
     <parent link="world" />

Commit message: ui working

File: vegebot_run/urdf/vegebot.urdf.xacro (robot description, xacro)
@@ -251,5 +251,5 @@
     <origin xyz="${-overhead_camera_support1_length + (overhead_camera_support2_width/2.0)} 0.0 ${overhead_camera_support2_width/2.0}" rpy="0.0 ${MPI/2.0} 0.0" />
   </joint>
-  <link name="overhead_camera">
+  <link name="overhead_camera_body">
     <visual>
       <geometry>
@@ -262,8 +262,15 @@
     </visual>
   </link>
-  <joint name="overhead_camera_support2_to_overhead_camera_joint" type="fixed">
+  <joint name="overhead_camera_support2_to_overhead_camera_body_joint" type="fixed">
     <parent link="overhead_camera_support2" />
+    <child link = "overhead_camera_body" />
+    <origin xyz="${-overhead_camera_support2_length + (overhead_camera_height/2.0)} 0.0 ${overhead_camera_support2_height/2.0 + overhead_camera_height/2.0}" rpy="0.0 ${MPI/2.0} 0.0" />
+  </joint>
+  <link name="overhead_camera">
+  </link>
+  <joint name="overhead_camera_body_to_overhead_camera_joint" type="fixed">
+    <parent link="overhead_camera_body" />
     <child link = "overhead_camera" />
-    <origin xyz="${-overhead_camera_support2_length + (overhead_camera_height/2.0)} 0.0 ${overhead_camera_support2_height/2.0 + overhead_camera_height/2.0}" rpy="0.0 ${MPI/2.0} 0.0" />
+    <origin xyz="0.0 0.0 0.0" rpy="${MPI + MPI/2.0} ${MPI} 0.0" />
   </joint>
   <joint name="world_joint" type="fixed">

Commit message: Model modified for Josies new end effector

File: vegebot_run/urdf/vegebot.urdf.xacro (robot description, xacro)
@@ -26,7 +26,9 @@
   <xacro:property name="wheel_length" value="0.10" />
   <xacro:property name="wheel_radius" value="0.20" />
-  <xacro:property name="bucket_length" value="0.24" />
+  <xacro:property name="bucket_length" value="0.29" />
   <xacro:property name="bucket_radius" value="0.14" />
   <xacro:property name="ee_bucket_offset_x" value="0.12" />
+  <xacro:property name="ee_bucket_offset_y" value="-0.13" />
+  <xacro:property name="ee_bucket_offset_z" value="0.0" />
   <xacro:property name="pneumatic_width" value="0.22" />
   <xacro:property name="pneumatic_depth" value="0.06" />
@@ -57,4 +59,5 @@
   <xacro:property name="overhead_camera_width" value="0.1" />
   <xacro:property name="overhead_camera_height" value="0.045" />
+  <xacro:property name="arm_to_overhead_camera_support1" value="0.43" />
   <xacro:macro name="wheel_assembly">
     <visual>
@@ -233,5 +236,5 @@
     <parent link="platform" />
     <child link = "overhead_camera_support1" />
-    <origin xyz="${-front_platform_to_origin_arm} 0.0 ${platform_height}" rpy="0.0 ${MPI/2.0} 0.0" />
+    <origin xyz="${-arm_to_overhead_camera_support1} 0.0 ${rear_platform_height}" rpy="0.0 ${MPI/2.0} 0.0" />
   </joint>
   <link name="overhead_camera_support2">
@@ -360,5 +363,5 @@
     <parent link="ee_link" />
     <child link = "bucket_link" />
-    <origin xyz="${ee_bucket_offset_x} 0.0 0.0" rpy="0.0 1.5708 0.0" />
+    <origin xyz="${ee_bucket_offset_x} ${ee_bucket_offset_y} ${ee_bucket_offset_z}" rpy="0.0 1.5708 0.0" />
   </joint>
   <link name="pneumatic_link">

Commit message: camera calibration files added

File: vegebot_run/urdf/vegebot.urdf.xacro (robot description, xacro)
@@ -347,5 +347,5 @@
     <parent link="ee_link" />
     <child link = "camera_link" />
-    <origin xyz="${bucket_length} ${-bucket_radius - camera_offset_z} 0.0" rpy="0.0 0.0 0.0" />
+    <origin xyz="${bucket_length*1.3} ${-bucket_radius - camera_offset_z} 0.0" rpy="0.0 0.0 0.0" />
   </joint>
   <link name="bucket_link">
@@ -363,5 +363,5 @@
     <parent link="ee_link" />
     <child link = "bucket_link" />
-    <origin xyz="${ee_bucket_offset_x} ${ee_bucket_offset_y} ${ee_bucket_offset_z}" rpy="0.0 1.5708 0.0" />
+    <origin xyz="${ee_bucket_offset_x*1.3} ${ee_bucket_offset_y} ${ee_bucket_offset_z}" rpy="0.0 1.5708 0.0" />
   </joint>
   <link name="pneumatic_link">

Commit message: Working with overhead camera

File: vegebot_run/urdf/vegebot.urdf.xacro (robot description, xacro)
@@ -275,5 +275,6 @@
     <parent link="overhead_camera_body" />
     <child link = "overhead_camera" />
-    <origin xyz="0.0 0.0 0.0" rpy="${MPI + MPI/2.0} ${MPI} 0.0" />
+    <!--  <origin xyz="0.0 0.0 0.0" rpy="${MPI + MPI/2.0} ${MPI} 0.0" /> -->
+    <origin xyz="0.0 0.0 0.0" rpy="0.0 ${MPI} 0.0" />
   </joint>
   <joint name="world_joint" type="fixed">

Commit message: tune for new  bucket

File: vegebot_run/urdf/vegebot.urdf.xacro (robot description, xacro)
@@ -9,5 +9,8 @@
   <xacro:property name="floor_thickness" value="0.05" />
   <xacro:property name="platform_width" value="2.12" />
+  <!--
   <xacro:property name="platform_height" value="0.58" />
+-->
+  <xacro:property name="platform_height" value="0.90" />
   <xacro:property name="platform_length" value="0.32" />
   <xacro:property name="platform_depth" value="0.10" />
@@ -28,7 +31,12 @@
   <xacro:property name="bucket_length" value="0.29" />
   <xacro:property name="bucket_radius" value="0.14" />
+  <xacro:property name="ee_bucket_offset_x" value="0.0" />
+  <xacro:property name="ee_bucket_offset_y" value="0.0" />
+  <xacro:property name="ee_bucket_offset_z" value="0.0" />
+  <!--
   <xacro:property name="ee_bucket_offset_x" value="0.12" />
   <xacro:property name="ee_bucket_offset_y" value="-0.13" />
   <xacro:property name="ee_bucket_offset_z" value="0.0" />
+  -->
   <xacro:property name="pneumatic_width" value="0.22" />
   <xacro:property name="pneumatic_depth" value="0.06" />

Commit message: calibrate

File: vegebot_run/urdf/vegebot.urdf.xacro (robot description, xacro)
@@ -5,4 +5,19 @@
   BIRL Laboratory, Engineering Dept., University of Cambridge
 -->
+  <!-- Lab or Platform -->
+  <xacro:property name="environment" value="lab" />
+  <!--
+  <xacro:property name="environment" value="platform" />
+  -->
+  <xacro:if value="${environment == 'lab'}">
+    <xacro:property name="arm_to_overhead_camera_support1" value="0.385" />
+    <xacro:property name="platform_height" value="0.90" />
+    <xacro:property name="rear_platform_to_overhead_camera_support1" value="${platform_height - rear_platform_height}" />
+  </xacro:if>
+  <xacro:if value="${environment == 'platform'}">
+    <xacro:property name="arm_to_overhead_camera_support1" value="0.43" />
+    <xacro:property name="platform_height" value="0.58" />
+    <xacro:property name="rear_platform_to_overhead_camera_support1" value="0.0" />
+  </xacro:if>
   <!-- Vegebot platform dimensions -->
   <xacro:property name="MPI" value="3.14159265359" />
@@ -10,7 +25,5 @@
   <xacro:property name="platform_width" value="2.12" />
   <!--
-  <xacro:property name="platform_height" value="0.58" />
 -->
-  <xacro:property name="platform_height" value="0.90" />
   <xacro:property name="platform_length" value="0.32" />
   <xacro:property name="platform_depth" value="0.10" />
@@ -64,8 +77,8 @@
   <xacro:property name="overhead_camera_support2_width" value="0.045" />
   <xacro:property name="overhead_camera_support2_height" value="0.045" />
-  <xacro:property name="overhead_camera_length" value="0.06" />
-  <xacro:property name="overhead_camera_width" value="0.1" />
-  <xacro:property name="overhead_camera_height" value="0.045" />
-  <xacro:property name="arm_to_overhead_camera_support1" value="0.43" />
+  <xacro:property name="overhead_camera_length" value="0.07" />
+  <xacro:property name="overhead_camera_width" value="0.01" />
+  <xacro:property name="overhead_camera_height" value="0.03" />
+  <xacro:property name="overhead_camera_offset" value="0.02" />
   <xacro:macro name="wheel_assembly">
     <visual>
@@ -235,5 +248,5 @@
         <box size="${overhead_camera_support1_length} ${overhead_camera_support1_width} ${overhead_camera_support1_height}" />
       </geometry>
-      <origin xyz="-0.6 0.0 0.0" />
+      <origin xyz="${-overhead_camera_support1_length / 2.0} 0.0 0.0" />
       <material name="gray">
          <color rgba="0.1 0.1 0.1 1" />
@@ -244,5 +257,5 @@
     <parent link="platform" />
     <child link = "overhead_camera_support1" />
-    <origin xyz="${-arm_to_overhead_camera_support1} 0.0 ${rear_platform_height}" rpy="0.0 ${MPI/2.0} 0.0" />
+    <origin xyz="${-arm_to_overhead_camera_support1} 0.0 ${rear_platform_height + rear_platform_to_overhead_camera_support1}" rpy="0.0 ${MPI/2.0} 0.0" />
   </joint>
   <link name="overhead_camera_support2">
@@ -265,5 +278,5 @@
     <visual>
       <geometry>
-        <box size="${overhead_camera_length} ${overhead_camera_width} ${overhead_camera_height}" />
+        <box size="${overhead_camera_height} ${overhead_camera_length} ${overhead_camera_width}" />
       </geometry>
       <origin xyz="${-overhead_camera_length/2.0} 0.0 0.0" />
@@ -276,5 +289,5 @@
     <parent link="overhead_camera_support2" />
     <child link = "overhead_camera_body" />
-    <origin xyz="${-overhead_camera_support2_length + (overhead_camera_height/2.0)} 0.0 ${overhead_camera_support2_height/2.0 + overhead_camera_height/2.0}" rpy="0.0 ${MPI/2.0} 0.0" />
+    <origin xyz="${-overhead_camera_support2_length + (overhead_camera_height/2.0)} ${overhead_camera_offset} ${overhead_camera_support2_height/2.0 + overhead_camera_width/2.0}" rpy="0.0 ${MPI/2.0} 0.0" />
   </joint>
   <link name="overhead_camera">
